File: microTouch-rounded.kicad_pcb (KiCad board)
At the start: 2 copper layers, 34.5 x 22.9 mm, 10 parts, among them J1 SERVO, J2 PRINTER, U1 A3144

Commit message: forgot to label the bins in the silk screen
Other:
- board text added: "5V"
- board text added: "GND"
- board text added: "SERVO"
- board text added: "SIG"
- board text added: "VSIG"
